File: hw/dash_cluster/carrier/carrier.kicad_sch (KiCad schematic)
At the start: 26 parts, among them J1 To display module, J2 Loom in, J3 Loom out, Q1 IRLML6402, U1 TSR 1-2450, U2 TJA1051T/3, U3 24LC256

Commit message: carrier: a schematic that shows its connections, and a board to go with it
The schematic drew every part with net labels on its pins and no wires at
all, which passed ERC and was unreadable. It is now three wired blocks -
the loom and the supply, CAN, the EEPROM - with power symbols and named
labels only where a net is worth naming.

Two things KiCad does quietly cost most of that work, and both are now
handled by the generator rather than by remembering them:

A wire ending part way along another connects only ONCE per wire, however
many junction dots are drawn, so one rail with four stubs read back with
three of them unconnected. Every wire is split into one segment per span.

A pin lying part way along a wire does not connect, but a wire whose corner
lands on a pin does - which had shorted SDA, SCL and TXD onto 3V3 at J1,
because three corners sat at their neighbours' y.

gen_pcb.py builds the board the same way: a placement table, four layers to
JLCPCB's rules, ground pours, and every pad's net taken from the schematic's
own exported netlist so the two cannot disagree. It checks itself twice -
KiCad's DRC with schematic parity, and a geometric pre-check that measures
each track and via against every pad it does not belong to, which caught the
12 V track running through the connector's mounting peg.

55 x 35 mm, grown from 45 x 30: the two right-angle Micro-Fits own 13.7 mm
of the left edge each, the socket 21.4 mm of the right, and U1 and C4 are
both over 12 mm wide. The supply chain and the short nets are routed; the
CAN pair and the four module signals are left for the interactive router,
which --check reports rather than hides.

Co-Authored-By: Claude Opus 5 (1M context) <noreply@anthropic.com>
Parts:
- added H1, H2, H3, H4: M2, MountingHole:MountingHole_2.2mm_M2, symbol Mechanical:MountingHole
- C7: value 4n7 (end only) -> 4n7
- J1: footprint Connector_PinHeader_2.54mm:PinHeader_1x08_P2.54mm_Vertical -> Connector_PinSocket_2.54mm:PinSocket_1x08_P2.54mm_Vertical
- J2, J3: footprint Connector_JST:JST_XH_B4B-XH-A_1x04_P2.50mm_Vertical -> Connector_Molex:Molex_Micro-Fit_3.0_43045-0400_2x02_P3.00mm_Horizontal
- R3, R4: value 60R4 (end only) -> 60R4
Connections:
- net CANH: now also D3.2 (A2); no longer D3.1 (A1)
- net CANL: now also D3.1 (A1); no longer D3.2 (A2)
- net GATE: now also R2.2; no longer R2.1
- net GND: now also D1.1 (A1), R2.1; no longer D1.2 (A2), R2.2
- net SCL: now also R6.2; no longer R6.1
- net SDA: now also R5.2; no longer R5.1
- net VIN: now also D1.2 (A2); no longer D1.1 (A1)
- net +12V_F renamed 12V_F
- net +12V_IN renamed +12V
- net 3V3 renamed +3V3
- net +3V3: now also R5.1, R6.1; no longer R5.2, R6.2
- net IO29_NC: no longer names the net of J1.1 (Pin_1)
Other:
- note added: "12 V IN, REVERSE POLARITY, 5 V"
- note added: "CAN"
- note added: "CONFIG EEPROM"
- note added: "R3, R4 and C7 are fitted ONLY on the two boards"
- note added: "at the ends of the bus - see schematic.txt"
- moved on the sheet: C1, C2, C3, C4, C5, C6, C7, C9, D1, D2, D3, D5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
